File: Kicad/FOC-driver.kicad_pcb (KiCad board)
At the start: 4 copper layers, 114 parts, among them CN1 XT30PW-M, J1 USB_C_Receptacle_USB2.0_16P, J10 Conn_01x01_Pin, J11 Conn_01x01_Pin, J15 OLED, J16 SWD, J18 Thermistor, J19 Ext. bulk, J2 HYG025N06LS1C2, J3 HYG025N06LS1C2, J4 HYG025N06LS1C2, J5 HYG025N06LS1C2, J6 HYG025N06LS1C2, J7 HYG025N06LS1C2, J8 CAN, J9 Conn_01x01_Pin, U1 USBLC6-2SC6, U2 SN65HVD230, U3 DRV8328ARUYR, U4 STM32G473RCTx, U5 AS5047P, U6 TLV75733PDBV, U7 LMR51610XDBVR, Y1 24MHz

Commit message: hw(stm32): changed MCU to STM32G431CBTx since opamps unused.
Parts:
- removed C1, C15, C2, C25, C3, C32, C34, C4, C44, C6, C9: 100n, Capacitor_SMD:C_0402_1005Metric
- removed C10, C11: 16p, Capacitor_SMD:C_0402_1005Metric
- removed C12, C13, C14, C16, C33: 10n, Capacitor_SMD:C_0402_1005Metric
- removed C17, C35, C36, C7, C8: 1u, Capacitor_SMD:C_0603_1608Metric
- removed C18: 0.1u, Capacitor_SMD:C_0603_1608Metric
- removed C19, C20, C5: 10u, Capacitor_SMD:C_1206_3216Metric
- removed C21: 470n, Capacitor_SMD:C_0805_2012Metric
- removed C22, C23, C24: 100n, Capacitor_SMD:C_0805_2012Metric
- removed C26, C27: 100n, Capacitor_SMD:C_01005_0402Metric
- removed C29: 2u2, Capacitor_SMD:C_0805_2012Metric
- removed C30: 0.1u, Capacitor_SMD:C_0402_1005Metric
- removed C31: 22u, Capacitor_SMD:C_1206_3216Metric
- removed C37, C38, C39: 2u2, Capacitor_SMD:C_1206_3216Metric
- removed C41, C42, C43: 100n, Capacitor_SMD:C_0603_1608Metric
- removed CN1: XT30PW-M, addons:CONN-TH_XT30PW-M
- removed D1: SMAJ26A, Diode_SMD:D_SMA
- removed D10, D11, D8: GREEN, LED_SMD:LED_0603_1608Metric
- removed D9: RED, LED_SMD:LED_0603_1608Metric
- removed FB1, FB2: 120R, Inductor_SMD:L_0603_1608Metric
- removed J1: USB_C_Receptacle_USB2.0_16P, Connector_USB:USB_C_Receptacle_GCT_USB4105-xx-A_16P_TopMnt_Horizontal
- removed J10, J11, J9: Conn_01x01_Pin, Connector_Wire:SolderWirePad_1x01_SMD_4x8mm
- removed J15: OLED, Connector_PinSocket_2.54mm:PinSocket_1x04_P2.54mm_Vertical
- removed J16: SWD, Connector_PinSocket_1.27mm:PinSocket_2x03_P1.27mm_Vertical
- removed J18: Thermistor, addons:2p SolderWire Pad
- removed J19: Ext. bulk, addons:2p WireSolder 1.5mmID_2.5mmOD
- removed J2, J3, J4, J5, J6, J7: HYG025N06LS1C2, addons:HYG025N06LS1C2
- removed J8: CAN, TerminalBlock:TerminalBlock_Xinya_XY308-2.54-2P_1x02_P2.54mm_Horizontal
- removed L3: 33u, Inductor_SMD:L_10.4x10.4_H4.8
- removed R1, R2: 5k1, Resistor_SMD:R_0402_1005Metric
- removed R10, R11, R6, R7: 22, Resistor_SMD:R_0603_1608Metric
- removed R12, R13, R8, R9: 22k, Resistor_SMD:R_0603_1608Metric
- removed R14, R21, R3: 1mR, Resistor_SMD:R_2512_6332Metric
- removed R15, R22, R33, R36, R37, R5: 10k, Resistor_SMD:R_0402_1005Metric
- removed R16, R23, R34, R4: 1k, Resistor_SMD:R_0402_1005Metric
- removed R17, R18: 22, Resistor_SMD:R_01005_0402Metric
- removed R19, R20: 22k, Resistor_SMD:R_01005_0402Metric
- removed R24, R25: 60, Resistor_SMD:R_0603_1608Metric
- removed R27, R29, R40: 10k, Resistor_SMD:R_01005_0402Metric
- removed R28: 220, Resistor_SMD:R_01005_0402Metric
- removed R30: 22k1, Resistor_SMD:R_0402_1005Metric
- removed R31: 118k, Resistor_SMD:R_0402_1005Metric
- removed R32: 330, Resistor_SMD:R_0603_1608Metric
- removed R35: 100k, Resistor_SMD:R_0402_1005Metric
- removed R38, R39: 220, Resistor_SMD:R_0603_1608Metric
- removed R41: 1k, Resistor_SMD:R_01005_0402Metric
- removed U1: USBLC6-2SC6, Package_TO_SOT_SMD:SOT-23-6
- removed U2: SN65HVD230, Package_SO:SOIC-8_3.9x4.9mm_P1.27mm
- removed U3: DRV8328ARUYR, addons:QFN-28_L4.0-W4.0-P0.40-BL-EP2.6 DRV8328
- removed U4: STM32G473RCTx, Package_QFP:LQFP-64_10x10mm_P0.5mm
- removed U5: AS5047P, Package_SO:TSSOP-14_4.4x5mm_P0.65mm
- removed U6: TLV75733PDBV, Package_TO_SOT_SMD:SOT-23-5
- removed U7: LMR51610XDBVR, Package_TO_SOT_SMD:SOT-23-6
- removed Y1: 24MHz, Crystal:Crystal_SMD_3225-4Pin_3.2x2.5mm

Commit message: hw(pcb): initial grouping + layout guidlines
Parts:
- added C1: 10u, Capacitor_SMD:C_1206_3216Metric, F.Cu at (172.2, 76.2)
- added C10: 100n, Capacitor_SMD:C_01005_0402Metric, F.Cu at (130.4, 102.5)
- added C11: 16p, Capacitor_SMD:C_0402_1005Metric, F.Cu at (159.0, 80.2)
- added C12: 16p, Capacitor_SMD:C_0402_1005Metric, F.Cu at (159.0, 82.5)
- added C13: 100n, Capacitor_SMD:C_0402_1005Metric, F.Cu at (115.1, 103.5)
- added C14: 1u, Capacitor_SMD:C_0603_1608Metric, F.Cu at (138.2, 114.7)
- added C15: 100n, Capacitor_SMD:C_0603_1608Metric, F.Cu at (95.5, 63.7)
- added C16: 2u2, Capacitor_SMD:C_1206_3216Metric, F.Cu at (119.9, 73.6)
- added C17: 100n, Capacitor_SMD:C_0603_1608Metric, F.Cu at (95.5, 66.2)
- added C18: 10n, Capacitor_SMD:C_0402_1005Metric, F.Cu at (123.6, 63.4)
- added C19: 100n, Capacitor_SMD:C_0603_1608Metric, F.Cu at (95.5, 68.7)
- added C2: 100n, Capacitor_SMD:C_0402_1005Metric, F.Cu at (160.8, 78.7)
- added C20: 2u2, Capacitor_SMD:C_1206_3216Metric, F.Cu at (119.9, 77.0)
- added C21: 100n, Capacitor_SMD:C_0603_1608Metric, F.Cu at (95.5, 71.2)
- added C22: 10n, Capacitor_SMD:C_0402_1005Metric, F.Cu at (123.6, 65.4)
- added C23: 100n, Capacitor_SMD:C_0603_1608Metric, F.Cu at (95.5, 73.7)
- added C24: 2u2, Capacitor_SMD:C_1206_3216Metric, F.Cu at (119.9, 80.3)
- added C25: 100n, Capacitor_SMD:C_0603_1608Metric, F.Cu at (95.5, 76.2)
- added C26: 10n, Capacitor_SMD:C_0402_1005Metric, F.Cu at (123.6, 67.3)
- added C27: 0.1u, Capacitor_SMD:C_0603_1608Metric, F.Cu at (150.6, 92.5)
- added C28: 10u, Capacitor_SMD:C_1206_3216Metric, F.Cu at (145.8, 90.4)
- added C29: 10u, Capacitor_SMD:C_1206_3216Metric, F.Cu at (145.8, 93.7)
- added C3: 100n, Capacitor_SMD:C_0402_1005Metric, F.Cu at (171.5, 78.2)
- added C30: 100n, Capacitor_SMD:C_0402_1005Metric, F.Cu at (139.9, 101.7)
- added C31: 470n, Capacitor_SMD:C_0805_2012Metric, F.Cu at (140.7, 90.2)
- added C32: 100n, Capacitor_SMD:C_0805_2012Metric, F.Cu at (140.7, 93.2)
- added C33: 100n, Capacitor_SMD:C_0805_2012Metric, F.Cu at (140.7, 96.2)
- added C34: 100n, Capacitor_SMD:C_0805_2012Metric, F.Cu at (140.7, 99.2)
- added C35: 10n, Capacitor_SMD:C_0402_1005Metric, F.Cu at (101.0, 108.9)
- added C36: 100n, Capacitor_SMD:C_0402_1005Metric, F.Cu at (101.0, 110.8)
- added C37: 100n, Capacitor_SMD:C_0402_1005Metric, F.Cu at (101.0, 112.8)
- added C38: 2u2, Capacitor_SMD:C_0805_2012Metric, F.Cu at (104.6, 112.7)
- added C39: 100n, Capacitor_SMD:C_0402_1005Metric, F.Cu at (101.0, 114.8)
- added C4: 100n, Capacitor_SMD:C_0402_1005Metric, F.Cu at (163.8, 76.2)
- added C40: 22u, Capacitor_SMD:C_1206_3216Metric, F.Cu at (105.2, 109.5)
- added C41: 1u, Capacitor_SMD:C_0603_1608Metric, F.Cu at (101.6, 89.9)
- added C42: 1u, Capacitor_SMD:C_0603_1608Metric, F.Cu at (101.6, 92.4)
- added C43: 10n, Capacitor_SMD:C_0402_1005Metric, F.Cu at (145.3, 67.2)
- added C44: 100n, Capacitor_SMD:C_0402_1005Metric, F.Cu at (181.8, 83.2)
- added C47: 100n, Capacitor_SMD:C_0402_1005Metric, F.Cu at (181.8, 78.0)
- added C5: 100n, Capacitor_SMD:C_0402_1005Metric, F.Cu at (170.8, 86.5)
- added C6: 100n, Capacitor_SMD:C_0402_1005Metric, F.Cu at (168.2, 88.2)
- added C7: 1u, Capacitor_SMD:C_0603_1608Metric, F.Cu at (169.0, 90.0)
- added C8: 1u, Capacitor_SMD:C_0603_1608Metric, F.Cu at (161.2, 76.5)
- added C9: 100n, Capacitor_SMD:C_0402_1005Metric, F.Cu at (167.2, 88.2)
- added CN1: XT30PW-M, addons:CONN-TH_XT30PW-M, F.Cu at (92.3, 95.7)
- added D1: GREEN, LED_SMD:LED_0603_1608Metric, F.Cu at (133.9, 90.0)
- added D2: RED, LED_SMD:LED_0603_1608Metric, F.Cu at (150.6, 90.0)
- added D3: SMAJ26A, Diode_SMD:D_SMA, F.Cu at (103.6, 105.6)
- added D4: GREEN, LED_SMD:LED_0603_1608Metric, F.Cu at (108.9, 112.5)
- added FB1: 120R, Inductor_SMD:L_0603_1608Metric, F.Cu at (170.5, 88.2)
- added FB2: 120R, Inductor_SMD:L_0603_1608Metric, F.Cu at (101.6, 95.0)
- added J1: Thermistor, addons:2p SolderWire Pad, F.Cu at (134.0, 103.5)
- added J2: Conn_01x01_Pin, Connector_Wire:SolderWirePad_1x01_SMD_4x8mm, F.Cu at (108.3, 67.2)
- added J3: Conn_01x01_Pin, Connector_Wire:SolderWirePad_1x01_SMD_4x8mm, F.Cu at (113.8, 67.2)
- added J4: Conn_01x01_Pin, Connector_Wire:SolderWirePad_1x01_SMD_4x8mm, F.Cu at (119.4, 67.2)
- added J5: Ext. bulk, addons:2p WireSolder 1.5mmID_2.5mmOD, F.Cu at (103.6, 102.5)
- added J6: CAN, TerminalBlock:TerminalBlock_Xinya_XY308-2.54-2P_1x02_P2.54mm_Horizontal, F.Cu at (150.8, 66.0)
- added J7: USB_C_Receptacle_USB2.0_16P, Connector_USB:USB_C_Receptacle_GCT_USB4105-xx-A_16P_TopMnt_Horizontal, F.Cu at (187.8, 80.8)
- added J8: SWD, Connector_PinSocket_1.27mm:PinSocket_2x03_P1.27mm_Vertical, F.Cu at (166.0, 71.7)
- added J9: OLED, Connector_PinSocket_2.54mm:PinSocket_1x04_P2.54mm_Vertical, F.Cu at (163.2, 68.2)
- added L1: 33u, Inductor_SMD:L_10.4x10.4_H4.8, F.Cu at (91.3, 110.5)
- added Q1: HYG025N06LS1C2, addons:HYG025N06LS1C2, F.Cu at (88.5, 58.2)
- added Q2: HYG025N06LS1C2, addons:HYG025N06LS1C2, F.Cu at (95.2, 58.2)
- added Q3: HYG025N06LS1C2, addons:HYG025N06LS1C2, F.Cu at (101.9, 58.2)
- added Q4: HYG025N06LS1C2, addons:HYG025N06LS1C2, F.Cu at (108.5, 58.2)
- added Q5: HYG025N06LS1C2, addons:HYG025N06LS1C2, F.Cu at (115.2, 58.2)
- added Q6: HYG025N06LS1C2, addons:HYG025N06LS1C2, F.Cu at (121.9, 58.2)
- added R1: 10k, Resistor_SMD:R_0402_1005Metric, F.Cu at (133.3, 92.3)
- added R10: 10k, Resistor_SMD:R_0402_1005Metric, F.Cu at (115.6, 72.9)
- added R11: 1k, Resistor_SMD:R_0402_1005Metric, F.Cu at (115.6, 74.9)
- added R12: 22, Resistor_SMD:R_0603_1608Metric, F.Cu at (99.5, 71.2)
- added R13: 22k, Resistor_SMD:R_0603_1608Metric, F.Cu at (99.5, 73.7)
- added R14: 5mR, Resistor_SMD:R_2512_6332Metric, F.Cu at (109.8, 79.3)
- added R15: 22, Resistor_SMD:R_0603_1608Metric, F.Cu at (99.5, 76.2)
- added R16: 22k, Resistor_SMD:R_0603_1608Metric, F.Cu at (99.5, 78.7)
- added R17: 10k, Resistor_SMD:R_0402_1005Metric, F.Cu at (115.6, 76.9)
- added R18: 1k, Resistor_SMD:R_0402_1005Metric, F.Cu at (115.6, 78.9)
- added R19: 22, Resistor_SMD:R_0603_1608Metric, F.Cu at (103.5, 63.7)
- added R2: 220, Resistor_SMD:R_0603_1608Metric, F.Cu at (118.5, 100.0)
- added R20: 22k, Resistor_SMD:R_0603_1608Metric, F.Cu at (103.5, 66.2)
- added R21: 5mR, Resistor_SMD:R_2512_6332Metric, F.Cu at (109.8, 84.2)
- added R22: 22, Resistor_SMD:R_0603_1608Metric, F.Cu at (103.5, 68.7)
- added R23: 22k, Resistor_SMD:R_0603_1608Metric, F.Cu at (103.5, 71.2)
- added R24: 10k, Resistor_SMD:R_0402_1005Metric, F.Cu at (115.6, 80.9)
- added R25: 1k, Resistor_SMD:R_0402_1005Metric, F.Cu at (115.6, 82.9)
- added R26: 10k, Resistor_SMD:R_01005_0402Metric, F.Cu at (150.4, 96.2)
- added R27: 100k, Resistor_SMD:R_0402_1005Metric, F.Cu at (150.8, 101.3)
- added R28: 10k, Resistor_SMD:R_01005_0402Metric, F.Cu at (150.4, 97.9)
- added R29: 220, Resistor_SMD:R_01005_0402Metric, F.Cu at (150.4, 99.5)
- added R3: 10k, Resistor_SMD:R_01005_0402Metric, F.Cu at (130.4, 104.2)
- added R30: 10k, Resistor_SMD:R_0402_1005Metric, F.Cu at (105.0, 89.7)
- added R31: 1k, Resistor_SMD:R_0402_1005Metric, F.Cu at (105.0, 91.7)
- added R32: 22k1, Resistor_SMD:R_0402_1005Metric, F.Cu at (105.0, 93.7)
- added R33: 118k, Resistor_SMD:R_0402_1005Metric, F.Cu at (105.0, 95.6)
- added R34: 10k, Resistor_SMD:R_0402_1005Metric, F.Cu at (105.0, 97.6)
- added R35: 220, Resistor_SMD:R_0603_1608Metric, F.Cu at (101.6, 97.5)
- added R36: 60, Resistor_SMD:R_0603_1608Metric, F.Cu at (142.3, 66.2)
- added R37: 60, Resistor_SMD:R_0603_1608Metric, F.Cu at (142.3, 68.5)
- added R38: 5k1, Resistor_SMD:R_0402_1005Metric, F.Cu at (181.7, 82.2)
- added R39: 5k1, Resistor_SMD:R_0402_1005Metric, F.Cu at (181.7, 79.0)
- added R4: 1k, Resistor_SMD:R_01005_0402Metric, F.Cu at (130.4, 105.8)
- added R5: 22, Resistor_SMD:R_0603_1608Metric, F.Cu at (95.5, 78.7)
- added R6: 22k, Resistor_SMD:R_0603_1608Metric, F.Cu at (99.5, 63.7)
- added R7: 5mR, Resistor_SMD:R_2512_6332Metric, F.Cu at (109.8, 74.4)
- added R8: 22, Resistor_SMD:R_0603_1608Metric, F.Cu at (99.5, 66.2)
- added R9: 22k, Resistor_SMD:R_0603_1608Metric, F.Cu at (99.5, 68.7)
- added U1: STM32G431C8Tx, Package_QFP:LQFP-48_7x7mm_P0.5mm, F.Cu at (166.5, 82.0)
- added U10: USBLC6-2SC6, Package_TO_SOT_SMD:SOT-23-6, F.Cu at (178.1, 80.5)
- added U2: AS5047P, Package_SO:TSSOP-14_4.4x5mm_P0.65mm, F.Cu at (133.0, 116.2)
- added U3: INA240A1D, Package_SO:SOIC-8_3.9x4.9mm_P1.27mm, F.Cu at (89.2, 65.8)
- added U4: INA240A1D, Package_SO:SOIC-8_3.9x4.9mm_P1.27mm, F.Cu at (89.2, 72.3)
- added U5: INA240A1D, Package_SO:SOIC-8_3.9x4.9mm_P1.27mm, F.Cu at (89.2, 78.9)
- added U6: DRV8328ARUYR, addons:QFN-28_L4.0-W4.0-P0.40-BL-EP2.6 DRV8328, F.Cu at (146.2, 98.5)
- added U7: LMR51610XDBVR, Package_TO_SOT_SMD:SOT-23-6, F.Cu at (114.2, 91.0)
- added U8: TLV75733PDBV, Package_TO_SOT_SMD:SOT-23-5, F.Cu at (109.0, 95.7)
- added U9: SN65HVD230, Package_SO:SOIC-8_3.9x4.9mm_P1.27mm, F.Cu at (136.5, 67.3)
- added Y1: 24MHz, Crystal:Crystal_SMD_3225-4Pin_3.2x2.5mm, F.Cu at (156.7, 81.3)

Commit message: commit
Parts:
- added C48: 100n, Capacitor_SMD:C_0402_1005Metric, F.Cu at (206.4, 97.4)
- added C49: 1u, Capacitor_SMD:C_0402_1005Metric, F.Cu at (207.4, 97.4)
- added D5: PESD1CAN,215, addons:PESD1CAN, F.Cu at (193.9, 97.4)
- added R40: 10k, Resistor_SMD:R_0402_1005Metric, B.Cu at (154.5, 97.2)
- added R41: 10k, Resistor_SMD:R_0402_1005Metric, F.Cu at (185.5, 75.0)
- C14, C43, R36, R37, U2: moved to B.Cu
- J2, J3, J4: footprint Connector_Wire:SolderWirePad_1x01_SMD_4x8mm -> addons:WireSolder-ID1.6mm-OD3mm
- J5: footprint addons:2p WireSolder 1.5mmID_2.5mmOD -> addons:2p WireSolder 1.3mmID_2mmOD
- R26, R28, R3, R4: footprint Resistor_SMD:R_01005_0402Metric -> Resistor_SMD:R_0402_1005Metric
- R29: footprint Resistor_SMD:R_01005_0402Metric -> Resistor_SMD:R_0603_1608Metric
- moved C13 116.8 mm to (230.7, 120.2)
- moved R35 110.5 mm to (210.0, 76.2)
- moved D4 110.4 mm to (214.0, 78.8)
- moved C42 108.1 mm to (208.8, 78.5)
- moved L1 104.0 mm to (191.8, 83.8)
- moved C41 100.2 mm to (200.8, 76.0)
- moved R34 97.7 mm to (200.8, 78.2)
- moved U8 97.4 mm to (204.8, 77.8)
- moved J1 96.7 mm to (229.7, 117.4)
- moved R3 96.1 mm to (225.8, 116.0)
- moved R4 96.1 mm to (225.8, 117.6)
- moved C40 95.2 mm to (194.6, 76.8), turned to 180 degrees
- moved C39 94.9 mm to (188.3, 77.8)
- moved R2 94.0 mm to (211.1, 116.2)
- moved C37 90.8 mm to (183.8, 75.5), turned to 180 degrees
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Connections:
- C37 pad 1: Net-(U7-EN) -> Net-(U7-VIN)
- C38 pad 1: Net-(U7-EN) -> Net-(U7-VIN)
- FB2 pad 2: Net-(U7-EN) -> Net-(U7-VIN)
- U2 pad 11: +5V -> unconnected-(U2-VDD-Pad11)
- U7 pad 1: LSS -> Net-(U7-CB)
- U7 pad 2: Net-(U7-SW) -> LSS
- U7 pad 3: Net-(U7-EN) -> Net-(U7-FB)
- U7 pad 4: Net-(U7-FB) -> Net-(U7-EN)
- U7 pad 5: Net-(U7-EN) -> Net-(U7-VIN)
- U7 pad 6: Net-(U7-CB) -> Net-(U7-SW)
Other:
- board outline added: 50 x 50 mm
