File: Kicad/comms.kicad_sch (KiCad schematic)
At the start: 14 parts, among them J1 USB_C_Receptacle_USB2.0_16P, J12 SPI1, J13 I2C1, J15 OLED, J16 SWD, J8 CAN, U1 USBLC6-2SC6, U2 SN65HVD230

Commit message: hw(pcb): initial grouping + layout guidlines
Parts:
- added C47: 100n, Capacitor_SMD:C_0402_1005Metric, symbol Device:C_Small
- renumbered C16 to C43, C9 to C44, J12 to J10, J13 to J11, J8 to J6, J1 to J7, J16 to J8, J15 to J9, R24 to R36, R25 to R37, R1 to R38, R2 to R39, U1 to U10, U2 to U9
Connections:
- net +5V: now also C47.1
- net GND: now also C47.2
- net USB_D+: now also J7.A6 (D+), J7.B6 (D+), U10.3 (I/O2)
- net USB_D-: now also J7.A7 (D-), J7.B7 (D-), U10.1 (I/O1)
Changed lines of the file:
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@@
 	)
 	(junction
+		(at 96.52 97.79)
+		(diameter 0)
+		(color 0 0 0 0)
+	)
+	(junction
 		(at 226.06 93.98)
 		(diameter 0)
@@
 	(wire
 		(pts
+			(xy 105.41 90.17) (xy 96.52 90.17)
+		)
+		(stroke
+			(width 0)
+			(type default)
+		)
+	)
+	(wire
+		(pts
 			(xy 213.36 130.81) (xy 213.36 129.54)
 		)
@@
 	(wire
 		(pts
+			(xy 105.41 97.79) (xy 96.52 97.79)
+		)
+		(stroke
+			(width 0)
+			(type default)
+		)
+	)
+	(wire
+		(pts
 			(xy 85.09 48.26) (xy 96.52 48.26)
 		)
@@
 	(wire
 		(pts
+			(xy 96.52 99.06) (xy 96.52 97.79)
+		)
+		(stroke
+			(width 0)
+			(type default)
+		)
+	)
+	(wire
+		(pts
 			(xy 58.42 66.04) (xy 69.85 66.04)
 		)
@@
 	(wire
 		(pts
+			(xy 105.41 96.52) (xy 105.41 97.79)
+		)
+		(stroke
+			(width 0)
+			(type default)
+		)
+	)
+	(wire
+		(pts
 			(xy 77.47 102.87) (xy 78.74 102.87)
 		)
@@
 	(wire
 		(pts
+			(xy 105.41 91.44) (xy 105.41 90.17)
+		)
+		(stroke
+			(width 0)
+			(type default)
+		)
+	)
+	(wire
+		(pts
 			(xy 104.14 55.88) (xy 104.14 57.15)
 		)
@@
 		)
 	)
+	(label "USB_D+"
+		(at 80.01 107.95 0)
+		(effects
+			(font
+				(size 0.762 0.762)
+			)
+			(justify left bottom)
+		)
+	)
+	(label "USB_D-"
+		(at 80.01 105.41 0)
+		(effects
+			(font
+				(size 0.762 0.762)
+			)
+			(justify left bottom)
+		)
+	)
 	(global_label "I2C1_SCL"
 		(shape input)
@@
 		(in_pos_files yes)
 		(dnp no)
-		(property "Reference" "C16"
+		(property "Reference" "C43"
 			(at 99.06 52.832 90)
 			(show_name no)
@@
 			(project "FOC-driver"
 				(path "/1cfe65f9-f673-4819-b0fb-9ca652a1a340/b3797230-ef53-49ba-9bea-2caddfb6bddf"
-					(reference "C16")
+					(reference "C43")
 					(unit 1)
 				)
@@
 		(dnp no)
 		(fields_autoplaced yes)
-		(property "Reference" "C9"
+		(property "Reference" "C44"
 			(at 99.06 92.7162 0)
 			(show_name no)
@@
 			(project "FOC-driver"
 				(path "/1cfe65f9-f673-4819-b0fb-9ca652a1a340/b3797230-ef53-49ba-9bea-2caddfb6bddf"
-					(reference "C9")
+					(reference "C44")
 					(unit 1)
 				)
@@
 		(dnp no)
 		(fields_autoplaced yes)
-		(property "Reference" "J8"
+		(property "Reference" "J6"
 			(at 149.86 53.3399 0)
 			(show_name no)
@@
 			(project "FOC-driver"
 				(path "/1cfe65f9-f673-4819-b0fb-9ca652a1a340/b3797230-ef53-49ba-9bea-2caddfb6bddf"
-					(reference "J8")
+					(reference "J6")
 					(unit 1)
 				)
@@
 		(dnp no)
 		(fields_autoplaced yes)
-		(property "Reference" "J15"
+		(property "Reference" "J9"
 			(at 222.25 124.4599 0)
 			(show_name no)
@@
 			(project "FOC-driver"
 				(path "/1cfe65f9-f673-4819-b0fb-9ca652a1a340/b3797230-ef53-49ba-9bea-2caddfb6bddf"
-					(reference "J15")
+					(reference "J9")
 					(unit 1)
 				)
@@
 		(dnp no)
 		(fields_autoplaced yes)
-		(property "Reference" "J1"
+		(property "Reference" "J7"
 			(at 62.23 82.55 0)
 			(show_name no)
@@
 			(project "FOC-driver"
 				(path "/1cfe65f9-f673-4819-b0fb-9ca652a1a340/b3797230-ef53-49ba-9bea-2caddfb6bddf"
-					(reference "J1")
+					(reference "J7")
 					(unit 1)
 				)
@@
 	(symbol
 		(lib_id "power:GND")
-		(at 96.52 97.79 0)
+		(at 96.52 99.06 0)
 		(unit 1)
 		(body_style 1)
@@
 		(fields_autoplaced yes)
 		(property "Reference" "#PWR012"
-			(at 96.52 104.14 0)
+			(at 96.52 105.41 0)
 			(hide yes)
 			(show_name no)
@@
 		)
 		(property "Value" "GND"
-			(at 96.52 102.87 0)
+			(at 96.52 104.14 0)
 			(hide yes)
 			(show_name no)
@@
 		)
 		(property "Footprint" ""
-			(at 96.52 97.79 0)
+			(at 96.52 99.06 0)
 			(hide yes)
 			(show_name no)
@@
 		)
 		(property "Datasheet" ""
-			(at 96.52 97.79 0)
+			(at 96.52 99.06 0)
 			(hide yes)
 			(show_name no)
@@
 		)
 		(property "Description" "Power symbol creates a global label with name \"GND\" , ground"
-			(at 96.52 97.79 0)
+			(at 96.52 99.06 0)
 			(hide yes)
 			(show_name no)
@@
 		(in_pos_files yes)
 		(dnp no)
-		(property "Reference" "R24"
+		(property "Reference" "R36"
 			(at 90.17 51.816 90)
 			(show_name no)
@@
 			(project "FOC-driver"
 				(path "/1cfe65f9-f673-4819-b0fb-9ca652a1a340/b3797230-ef53-49ba-9bea-2caddfb6bddf"
-					(reference "R24")
+					(reference "R36")
 					(unit 1)
 				)
@@
 		(dnp yes)
 		(fields_autoplaced yes)
-		(property "Reference" "J13"
+		(property "Reference" "J11"
 			(at 153.67 123.1899 0)
 			(show_name no)
@@
 			(project "FOC-driver"
 				(path "/1cfe65f9-f673-4819-b0fb-9ca652a1a340/b3797230-ef53-49ba-9bea-2caddfb6bddf"
-					(reference "J13")
+					(reference "J11")
 					(unit 1)
 				)
@@
 		(dnp yes)
 		(fields_autoplaced yes)
-		(property "Reference" "J12"
+		(property "Reference" "J10"
 			(at 153.67 91.4399 0)
 			(show_name no)
@@
 			(project "FOC-driver"
 				(path "/1cfe65f9-f673-4819-b0fb-9ca652a1a340/b3797230-ef53-49ba-9bea-2caddfb6bddf"
-					(reference "J12")
+					(reference "J10")
 					(unit 1)
 				)
@@
 		(in_pos_files yes)
 		(dnp no)
-		(property "Reference" "R1"
+		(property "Reference" "R38"
 			(at 81.28 90.932 90)
 			(show_name no)
@@
 			(project "FOC-driver"
 				(path "/1cfe65f9-f673-4819-b0fb-9ca652a1a340/b3797230-ef53-49ba-9bea-2caddfb6bddf"
-					(reference "R1")
+					(reference "R38")
 					(unit 1)
 				)
@@
 	)
 	(symbol
+		(lib_id "Device:C_Small")
+		(at 105.41 93.98 0)
+		(unit 1)
+		(body_style 1)
+		(exclude_from_sim no)
+		(in_bom yes)
+		(on_board yes)
+		(in_pos_files yes)
+		(dnp no)
+		(fields_autoplaced yes)
+		(property "Reference" "C47"
+			(at 107.95 92.7162 0)
+			(show_name no)
+			(do_not_autoplace no)
+			(effects
+				(font
+					(size 1.27 1.27)
+				)
+				(justify left)
+			)
+		)
+		(property "Value" "100n"
+			(at 107.95 95.2562 0)
+			(show_name no)
+			(do_not_autoplace no)
+			(effects
+				(font
+					(size 1.27 1.27)
+				)
+				(justify left)
+			)
+		)
+		(property "Footprint" "Capacitor_SMD:C_0402_1005Metric"
+			(at 105.41 93.98 0)
+			(hide yes)
+			(show_name no)
+			(do_not_autoplace no)
+			(effects
+				(font
+					(size 1.27 1.27)
+				)
+			)
+		)
+		(property "Datasheet" ""
+			(at 105.41 93.98 0)
+			(hide yes)
+			(show_name no)
+			(do_not_autoplace no)
+			(effects
+				(font
+					(size 1.27 1.27)
+				)
+			)
+		)
+		(property "Description" "Unpolarized capacitor, small symbol"
+			(at 105.41 93.98 0)
+			(hide yes)
+			(show_name no)
+			(do_not_autoplace no)
+			(effects
+				(font
+					(size 1.27 1.27)
+				)
+			)
+		)
+		(pin "2"
+		)
+		(pin "1"
+		)
+		(instances
+			(project "FOC-driver"
+				(path "/1cfe65f9-f673-4819-b0fb-9ca652a1a340/b3797230-ef53-49ba-9bea-2caddfb6bddf"
+					(reference "C47")
+					(unit 1)
+				)
+			)
+		)
+	)
+	(symbol
 		(lib_id "Device:R_Small")
 		(at 81.28 97.79 90)
@@
 		(in_pos_files yes)
 		(dnp no)
-		(property "Reference" "R2"
+		(property "Reference" "R39"
 			(at 81.28 102.108 90)
 			(show_name no)
@@
 			(project "FOC-driver"
 				(path "/1cfe65f9-f673-4819-b0fb-9ca652a1a340/b3797230-ef53-49ba-9bea-2caddfb6bddf"
-					(reference "R2")
+					(reference "R39")
 					(unit 1)
 				)
@@
 		(in_pos_files yes)
 		(dnp no)
-		(property "Reference" "R25"
+		(property "Reference" "R37"
 			(at 90.17 56.896 90)
 			(show_name no)
@@
 			(project "FOC-driver"
 				(path "/1cfe65f9-f673-4819-b0fb-9ca652a1a340/b3797230-ef53-49ba-9bea-2caddfb6bddf"
-					(reference "R25")
+					(reference "R37")
 					(unit 1)
 				)
@@
 		(dnp no)
 		(fields_autoplaced yes)
-		(property "Reference" "J16"
+		(property "Reference" "J8"
 			(at 217.17 82.55 0)
 			(show_name no)
@@
 			(project "FOC-driver"
 				(path "/1cfe65f9-f673-4819-b0fb-9ca652a1a340/b3797230-ef53-49ba-9bea-2caddfb6bddf"
-					(reference "J16")
+					(reference "J8")
 					(unit 1)
 				)
@@
 		(in_pos_files yes)
 		(dnp no)
-		(property "Reference" "U2"
+		(property "Reference" "U9"
 			(at 74.93 63.754 0)
 			(show_name no)
@@
 			(project "FOC-driver"
 				(path "/1cfe65f9-f673-4819-b0fb-9ca652a1a340/b3797230-ef53-49ba-9bea-2caddfb6bddf"
-					(reference "U2")
+					(reference "U9")
 					(unit 1)
 				)
@@
 		(in_pos_files yes)
 		(dnp no)
-		(property "Reference" "U1"
+		(property "Reference" "U10"
 			(at 91.44 101.092 0)
 			(show_name no)
@@
 			(project "FOC-driver"
 				(path "/1cfe65f9-f673-4819-b0fb-9ca652a1a340/b3797230-ef53-49ba-9bea-2caddfb6bddf"
-					(reference "U1")
+					(reference "U10")
 					(unit 1)
 				)

Commit message: commit
Parts:
- added C48: 100n, Capacitor_SMD:C_0402_1005Metric, symbol Device:C_Small
- added C49: 1u, Capacitor_SMD:C_0402_1005Metric, symbol Device:C_Small
- added D5: PESD1CAN,215, addons:PESD1CAN, symbol component-addon:PESD1CAN,215
Connections:
- net +3.3V: now also C48.2, C49.2
- net CANH: now also D5.2
- net CANL: now also D5.1
- net GND: now also C48.1, C49.1, D5.3
Other:
- moved on the sheet: C43, J6, R36, R37, U9
