File: Kicad/driver.kicad_sch (KiCad schematic)
At the start: 14 parts, among them U3 DRV8328ARUYR

Commit message: hw(pcb): initial grouping + layout guidlines
Parts:
- renumbered C18 to C27, C19 to C28, C20 to C29, C25 to C30, C21 to C31, C22 to C32, C23 to C33, C24 to C34, D9 to D2, R27 to R26, R35 to R27, R29 to R28, R28 to R29, U3 to U6
Changed lines of the file:
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@@
 		(dnp no)
 		(fields_autoplaced yes)
-		(property "Reference" "C19"
+		(property "Reference" "C28"
 			(at 82.55 62.2362 0)
 			(show_name no)
@@
 			(project "FOC-driver"
 				(path "/1cfe65f9-f673-4819-b0fb-9ca652a1a340/4b7eaccf-cbdc-4b7c-9a55-ed2a1b3a214b"
-					(reference "C19")
+					(reference "C28")
 					(unit 1)
 				)
@@
 		(dnp no)
 		(fields_autoplaced yes)
-		(property "Reference" "C25"
+		(property "Reference" "C30"
 			(at 87.63 81.2862 0)
 			(show_name no)
@@
 			(project "FOC-driver"
 				(path "/1cfe65f9-f673-4819-b0fb-9ca652a1a340/4b7eaccf-cbdc-4b7c-9a55-ed2a1b3a214b"
-					(reference "C25")
+					(reference "C30")
 					(unit 1)
 				)
@@
 		(in_pos_files yes)
 		(dnp no)
-		(property "Reference" "R27"
+		(property "Reference" "R26"
 			(at 151.384 60.198 90)
 			(show_name no)
@@
 			(project "FOC-driver"
 				(path "/1cfe65f9-f673-4819-b0fb-9ca652a1a340/4b7eaccf-cbdc-4b7c-9a55-ed2a1b3a214b"
-					(reference "R27")
+					(reference "R26")
 					(unit 1)
 				)
@@
 		(dnp no)
 		(fields_autoplaced yes)
-		(property "Reference" "C20"
+		(property "Reference" "C29"
 			(at 78.74 81.2862 0)
 			(show_name no)
@@
 			(project "FOC-driver"
 				(path "/1cfe65f9-f673-4819-b0fb-9ca652a1a340/4b7eaccf-cbdc-4b7c-9a55-ed2a1b3a214b"
-					(reference "C20")
+					(reference "C29")
 					(unit 1)
 				)
@@
 		(in_pos_files yes)
 		(dnp no)
-		(property "Reference" "R29"
+		(property "Reference" "R28"
 			(at 223.012 74.676 0)
 			(show_name no)
@@
 			(project "FOC-driver"
 				(path "/1cfe65f9-f673-4819-b0fb-9ca652a1a340/4b7eaccf-cbdc-4b7c-9a55-ed2a1b3a214b"
-					(reference "R29")
+					(reference "R28")
 					(unit 1)
 				)
@@
 		(dnp no)
 		(fields_autoplaced yes)
-		(property "Reference" "C24"
+		(property "Reference" "C34"
 			(at 191.77 110.4962 0)
 			(show_name no)
@@
 			(project "FOC-driver"
 				(path "/1cfe65f9-f673-4819-b0fb-9ca652a1a340/4b7eaccf-cbdc-4b7c-9a55-ed2a1b3a214b"
-					(reference "C24")
+					(reference "C34")
 					(unit 1)
 				)
@@
 		(dnp no)
 		(fields_autoplaced yes)
-		(property "Reference" "U3"
+		(property "Reference" "U6"
 			(at 124.46 91.44 0)
 			(show_name no)
@@
 			(project "FOC-driver"
 				(path "/1cfe65f9-f673-4819-b0fb-9ca652a1a340/4b7eaccf-cbdc-4b7c-9a55-ed2a1b3a214b"
-					(reference "U3")
+					(reference "U6")
 					(unit 1)
 				)
@@
 		(dnp no)
 		(fields_autoplaced yes)
-		(property "Reference" "C18"
+		(property "Reference" "C27"
 			(at 73.66 62.2362 0)
 			(show_name no)
@@
 			(project "FOC-driver"
 				(path "/1cfe65f9-f673-4819-b0fb-9ca652a1a340/4b7eaccf-cbdc-4b7c-9a55-ed2a1b3a214b"
-					(reference "C18")
+					(reference "C27")
 					(unit 1)
 				)
@@
 		(dnp no)
 		(fields_autoplaced yes)
-		(property "Reference" "C22"
+		(property "Reference" "C32"
 			(at 152.4 110.4962 0)
 			(show_name no)
@@
 			(project "FOC-driver"
 				(path "/1cfe65f9-f673-4819-b0fb-9ca652a1a340/4b7eaccf-cbdc-4b7c-9a55-ed2a1b3a214b"
-					(reference "C22")
+					(reference "C32")
 					(unit 1)
 				)
@@
 		(in_pos_files yes)
 		(dnp no)
-		(property "Reference" "D9"
+		(property "Reference" "D2"
 			(at 237.236 72.39 90)
 			(show_name no)
@@
 			(project "FOC-driver"
 				(path "/1cfe65f9-f673-4819-b0fb-9ca652a1a340/4b7eaccf-cbdc-4b7c-9a55-ed2a1b3a214b"
-					(reference "D9")
+					(reference "D2")
 					(unit 1)
 				)
@@
 		(dnp no)
 		(fields_autoplaced yes)
-		(property "Reference" "C21"
+		(property "Reference" "C31"
 			(at 130.81 110.4962 0)
 			(show_name no)
@@
 			(project "FOC-driver"
 				(path "/1cfe65f9-f673-4819-b0fb-9ca652a1a340/4b7eaccf-cbdc-4b7c-9a55-ed2a1b3a214b"
-					(reference "C21")
+					(reference "C31")
 					(unit 1)
 				)
@@
 		(dnp no)
 		(fields_autoplaced yes)
-		(property "Reference" "C23"
+		(property "Reference" "C33"
 			(at 172.72 110.4962 0)
 			(show_name no)
@@
 			(project "FOC-driver"
 				(path "/1cfe65f9-f673-4819-b0fb-9ca652a1a340/4b7eaccf-cbdc-4b7c-9a55-ed2a1b3a214b"
-					(reference "C23")
+					(reference "C33")
 					(unit 1)
 				)
@@
 		(in_pos_files yes)
 		(dnp no)
-		(property "Reference" "R35"
+		(property "Reference" "R27"
 			(at 169.418 72.136 90)
 			(show_name no)
@@
 			(project "FOC-driver"
 				(path "/1cfe65f9-f673-4819-b0fb-9ca652a1a340/4b7eaccf-cbdc-4b7c-9a55-ed2a1b3a214b"
-					(reference "R35")
+					(reference "R27")
 					(unit 1)
 				)
@@
 		(in_pos_files yes)
 		(dnp no)
-		(property "Reference" "R28"
+		(property "Reference" "R29"
 			(at 231.394 72.898 90)
 			(show_name no)
@@
 			(project "FOC-driver"
 				(path "/1cfe65f9-f673-4819-b0fb-9ca652a1a340/4b7eaccf-cbdc-4b7c-9a55-ed2a1b3a214b"
-					(reference "R28")
-					(unit 1)
-				)
+					(reference "R29")
+					(unit 1)
+				)

Commit message: commit
Parts:
- R26, R28: footprint Resistor_SMD:R_01005_0402Metric -> Resistor_SMD:R_0402_1005Metric
- R29: footprint Resistor_SMD:R_01005_0402Metric -> Resistor_SMD:R_0603_1608Metric
Changed lines of the file:
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@@
 			)
 		)
-		(property "Footprint" "Resistor_SMD:R_01005_0402Metric"
+		(property "Footprint" "Resistor_SMD:R_0402_1005Metric"
 			(at 149.86 55.88 0)
 			(hide yes)
@@
 			)
 		)
-		(property "Footprint" "Resistor_SMD:R_01005_0402Metric"
+		(property "Footprint" "Resistor_SMD:R_0402_1005Metric"
 			(at 224.79 73.66 0)
 			(hide yes)
@@
 			)
 		)
-		(property "Footprint" "Resistor_SMD:R_01005_0402Metric"
+		(property "Footprint" "Resistor_SMD:R_0603_1608Metric"
 			(at 229.87 68.58 0)
 			(hide yes)
