File: Kicad/half-bridges.kicad_sch (KiCad schematic)
At the start: 45 parts, among them J10 Conn_01x01_Pin, J11 Conn_01x01_Pin, J14 HYG025N06LS1C2, J17 HYG025N06LS1C2, J2 HYG025N06LS1C2, J20 HYG025N06LS1C2, J21 HYG025N06LS1C2, J3 HYG025N06LS1C2, J9 Conn_01x01_Pin, U10 INA240A1D, U8 INA240A1D, U9 INA240A1D

Commit message: hw(pcb-sch): rename component ref & pcb manufacturing capability
Parts:
- renumbered C41 to C15, C37 to C16, C46 to C17, C12 to C18, C45 to C19, C47 to C20, C48 to C21, C49 to C22, C50 to C23, C51 to C24, C52 to C25, C53 to C26, J2 to J1, J3 to J2, J9 to J2, J10 to J3, J14 to J3, J11 to J4, J17 to J4, J20 to J5, J21 to J6, R5 to R10, R4 to R11, R26 to R12, R43 to R13, R47 to R14, R42 to R15, R44 to R16, R45 to R17, R46 to R18, R48 to R19, R50 to R20, R54 to R21, R49 to R22, R51 to R23, R52 to R24, R53 to R25, R6 to R5, R8 to R6, R3 to R7, R7 to R8

Commit message: hw(pcb): initial grouping + layout guidlines
Parts:
- renumbered J1 to Q1, J2 to Q2, J3 to Q3, J4 to Q4, J5 to Q5, J6 to Q6, U8 to U3, U9 to U4, U10 to U5
Changed lines of the file:
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@@
 	)
 	(symbol
-		(lib_name "HYG025N06LS1C2_1")
 		(lib_id "component-addon:HYG025N06LS1C2")
 		(at 82.55 44.45 0)
@@
 		(in_pos_files yes)
 		(dnp no)
-		(property "Reference" "J1"
+		(property "Reference" "Q1"
 			(at 91.44 39.3699 0)
 			(show_name no)
@@
 		(pin "1"
 		)
-		(pin "7"
+		(pin "8"
 		)
 		(pin "3"
@@
 		(pin "5"
 		)
-		(pin "6"
+		(pin "7"
 		)
 		(pin "2"
 		)
-		(pin "8"
+		(pin "6"
 		)
 		(instances
 			(project "FOC-driver"
 				(path "/1cfe65f9-f673-4819-b0fb-9ca652a1a340/248405ad-1825-484c-82f9-c319ebcf1726"
-					(reference "J1")
+					(reference "Q1")
 					(unit 1)
 				)
@@
 	)
 	(symbol
-		(lib_name "HYG025N06LS1C2_1")
 		(lib_id "component-addon:HYG025N06LS1C2")
 		(at 179.07 44.45 0)
@@
 		(in_pos_files yes)
 		(dnp no)
-		(property "Reference" "J3"
+		(property "Reference" "Q3"
 			(at 187.96 39.3699 0)
 			(show_name no)
@@
 			(project "FOC-driver"
 				(path "/1cfe65f9-f673-4819-b0fb-9ca652a1a340/248405ad-1825-484c-82f9-c319ebcf1726"
-					(reference "J3")
+					(reference "Q3")
 					(unit 1)
 				)
@@
 	)
 	(symbol
-		(lib_name "HYG025N06LS1C2_1")
 		(lib_id "component-addon:HYG025N06LS1C2")
 		(at 82.55 64.77 0)
@@
 		(in_pos_files yes)
 		(dnp no)
-		(property "Reference" "J2"
+		(property "Reference" "Q2"
 			(at 91.44 59.6899 0)
 			(show_name no)
@@
 		(pin "1"
 		)
-		(pin "7"
+		(pin "6"
 		)
 		(pin "3"
@@
 		(pin "5"
 		)
-		(pin "6"
+		(pin "8"
 		)
 		(pin "2"
 		)
-		(pin "8"
+		(pin "7"
 		)
 		(instances
 			(project "FOC-driver"
 				(path "/1cfe65f9-f673-4819-b0fb-9ca652a1a340/248405ad-1825-484c-82f9-c319ebcf1726"
-					(reference "J2")
+					(reference "Q2")
 					(unit 1)
 				)
@@
 	)
 	(symbol
-		(lib_name "HYG025N06LS1C2_1")
 		(lib_id "component-addon:HYG025N06LS1C2")
 		(at 82.55 138.43 0)
@@
 		(in_pos_files yes)
 		(dnp no)
-		(property "Reference" "J6"
+		(property "Reference" "Q6"
 			(at 91.44 133.3499 0)
 			(show_name no)
@@
 		(pin "1"
 		)
-		(pin "7"
+		(pin "8"
 		)
 		(pin "3"
@@
 		(pin "5"
 		)
-		(pin "6"
+		(pin "7"
 		)
 		(pin "2"
 		)
-		(pin "8"
+		(pin "6"
 		)
 		(instances
 			(project "FOC-driver"
 				(path "/1cfe65f9-f673-4819-b0fb-9ca652a1a340/248405ad-1825-484c-82f9-c319ebcf1726"
-					(reference "J6")
+					(reference "Q6")
 					(unit 1)
 				)
@@
 		(in_pos_files yes)
 		(dnp no)
-		(property "Reference" "U10"
+		(property "Reference" "U5"
 			(at 124.46 137.922 90)
 			(show_name no)
@@
 			(project "FOC-driver"
 				(path "/1cfe65f9-f673-4819-b0fb-9ca652a1a340/248405ad-1825-484c-82f9-c319ebcf1726"
-					(reference "U10")
+					(reference "U5")
 					(unit 1)
 				)
@@
 	)
 	(symbol
-		(lib_name "HYG025N06LS1C2_1")
 		(lib_id "component-addon:HYG025N06LS1C2")
 		(at 179.07 64.77 0)
@@
 		(in_pos_files yes)
 		(dnp no)
-		(property "Reference" "J4"
+		(property "Reference" "Q4"
 			(at 187.96 59.6899 0)
 			(show_name no)
@@
 			(project "FOC-driver"
 				(path "/1cfe65f9-f673-4819-b0fb-9ca652a1a340/248405ad-1825-484c-82f9-c319ebcf1726"
-					(reference "J4")
+					(reference "Q4")
 					(unit 1)
 				)
@@
 		(in_pos_files yes)
 		(dnp no)
-		(property "Reference" "U8"
+		(property "Reference" "U3"
 			(at 124.46 64.262 90)
 			(show_name no)
@@
 			(project "FOC-driver"
 				(path "/1cfe65f9-f673-4819-b0fb-9ca652a1a340/248405ad-1825-484c-82f9-c319ebcf1726"
-					(reference "U8")
+					(reference "U3")
 					(unit 1)
 				)
@@
 	)
 	(symbol
-		(lib_name "HYG025N06LS1C2_1")
 		(lib_id "component-addon:HYG025N06LS1C2")
 		(at 82.55 118.11 0)
@@
 		(in_pos_files yes)
 		(dnp no)
-		(property "Reference" "J5"
+		(property "Reference" "Q5"
 			(at 91.44 113.0299 0)
 			(show_name no)
@@
 		(pin "1"
 		)
-		(pin "7"
+		(pin "6"
 		)
 		(pin "3"
@@
 		(pin "5"
 		)
-		(pin "6"
+		(pin "7"
 		)
 		(pin "2"
@@
 			(project "FOC-driver"
 				(path "/1cfe65f9-f673-4819-b0fb-9ca652a1a340/248405ad-1825-484c-82f9-c319ebcf1726"
-					(reference "J5")
+					(reference "Q5")
 					(unit 1)
 				)
@@
 		(in_pos_files yes)
 		(dnp no)
-		(property "Reference" "U9"
+		(property "Reference" "U4"
 			(at 220.98 64.262 90)
 			(show_name no)
@@
 			(project "FOC-driver"
 				(path "/1cfe65f9-f673-4819-b0fb-9ca652a1a340/248405ad-1825-484c-82f9-c319ebcf1726"
-					(reference "U9")
+					(reference "U4")
 					(unit 1)
 				)

Commit message: commit
Parts:
- J2, J3, J4: footprint Connector_Wire:SolderWirePad_1x01_SMD_4x8mm -> addons:WireSolder-ID1.6mm-OD3mm
Changed lines of the file:
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@@
 			)
 		)
-		(property "Footprint" "Connector_Wire:SolderWirePad_1x01_SMD_4x8mm"
+		(property "Footprint" "addons:WireSolder-ID1.6mm-OD3mm"
 			(at 199.39 125.73 0)
 			(hide yes)
@@
 			)
 		)
-		(property "Footprint" "Connector_Wire:SolderWirePad_1x01_SMD_4x8mm"
+		(property "Footprint" "addons:WireSolder-ID1.6mm-OD3mm"
 			(at 199.39 135.89 0)
 			(hide yes)
@@
 			)
 		)
-		(property "Footprint" "Connector_Wire:SolderWirePad_1x01_SMD_4x8mm"
+		(property "Footprint" "addons:WireSolder-ID1.6mm-OD3mm"
 			(at 199.39 115.57 0)
 			(hide yes)
