File: Kicad/power.kicad_sch (KiCad schematic)
At the start: 24 parts, among them CN1 XT30PW-M, J19 Ext. bulk, U6 TLV75733PDBV, U7 LMR51610XDBVR

Commit message: hw(pcb-sch): rename component ref & pcb manufacturing capability
Parts:
- C30: value 0.1u -> 100n
Changed lines of the file:
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@@
 	(text "External bulk cap. bank\n4x 220/330uF, 63V"
 		(exclude_from_sim no)
-		(at 103.378 66.04 0)
+		(at 77.47 49.784 0)
 		(effects
 			(font
@@
 			)
 		)
-		(property "Value" "0.1u"
+		(property "Value" "100n"
 			(at 153.6636 82.55 90)
 			(show_name no)

Commit message: hw(pcb): initial grouping + layout guidlines
Parts:
- renumbered C33 to C35, C32 to C36, C34 to C37, C29 to C38, C30 to C39, C31 to C40, C35 to C41, C36 to C42, C28 to C45, C40 to C46, D1 to D3, D11 to D4, J19 to J5, L3 to L1, R33 to R30, R34 to R31, R30 to R32, R31 to R33, R36 to R34, R39 to R35, U6 to U8
Changed lines of the file:
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@@
 		(dnp no)
 		(fields_autoplaced yes)
-		(property "Reference" "C30"
+		(property "Reference" "C39"
 			(at 153.6636 80.01 90)
 			(show_name no)
@@
 			(project "FOC-driver"
 				(path "/1cfe65f9-f673-4819-b0fb-9ca652a1a340/f11b4b8c-1f7a-4164-8f83-b37924046d35"
-					(reference "C30")
+					(reference "C39")
 					(unit 1)
 				)
@@
 		(in_pos_files yes)
 		(dnp no)
-		(property "Reference" "C31"
+		(property "Reference" "C40"
 			(at 168.402 95.758 0)
 			(show_name no)
@@
 			(project "FOC-driver"
 				(path "/1cfe65f9-f673-4819-b0fb-9ca652a1a340/f11b4b8c-1f7a-4164-8f83-b37924046d35"
-					(reference "C31")
+					(reference "C40")
 					(unit 1)
 				)
@@
 		(dnp no)
 		(fields_autoplaced yes)
-		(property "Reference" "D1"
+		(property "Reference" "D3"
 			(at 54.61 93.9799 90)
 			(show_name no)
@@
 			(project "FOC-driver"
 				(path "/1cfe65f9-f673-4819-b0fb-9ca652a1a340/f11b4b8c-1f7a-4164-8f83-b37924046d35"
-					(reference "D1")
+					(reference "D3")
 					(unit 1)
 				)
@@
 		(in_pos_files yes)
 		(dnp no)
-		(property "Reference" "C32"
+		(property "Reference" "C36"
 			(at 97.282 94.488 0)
 			(show_name no)
@@
 			(project "FOC-driver"
 				(path "/1cfe65f9-f673-4819-b0fb-9ca652a1a340/f11b4b8c-1f7a-4164-8f83-b37924046d35"
-					(reference "C32")
+					(reference "C36")
 					(unit 1)
 				)
@@
 		(in_pos_files yes)
 		(dnp no)
-		(property "Reference" "C33"
+		(property "Reference" "C35"
 			(at 76.962 99.568 0)
 			(show_name no)
@@
 			(project "FOC-driver"
 				(path "/1cfe65f9-f673-4819-b0fb-9ca652a1a340/f11b4b8c-1f7a-4164-8f83-b37924046d35"
-					(reference "C33")
+					(reference "C35")
 					(unit 1)
 				)
@@
 		(dnp yes)
 		(fields_autoplaced yes)
-		(property "Reference" "C28"
+		(property "Reference" "C45"
 			(at 104.14 54.9909 0)
 			(show_name no)
@@
 			(project "FOC-driver"
 				(path "/1cfe65f9-f673-4819-b0fb-9ca652a1a340/f11b4b8c-1f7a-4164-8f83-b37924046d35"
-					(reference "C28")
+					(reference "C45")
 					(unit 1)
 				)
@@
 		(in_pos_files yes)
 		(dnp no)
-		(property "Reference" "R34"
+		(property "Reference" "R31"
 			(at 68.072 99.314 0)
 			(show_name no)
@@
 			(project "FOC-driver"
 				(path "/1cfe65f9-f673-4819-b0fb-9ca652a1a340/f11b4b8c-1f7a-4164-8f83-b37924046d35"
-					(reference "R34")
+					(reference "R31")
 					(unit 1)
 				)
@@
 		(in_pos_files yes)
 		(dnp no)
-		(property "Reference" "R30"
+		(property "Reference" "R32"
 			(at 149.606 96.774 0)
 			(show_name no)
@@
 			(project "FOC-driver"
 				(path "/1cfe65f9-f673-4819-b0fb-9ca652a1a340/f11b4b8c-1f7a-4164-8f83-b37924046d35"
-					(reference "R30")
+					(reference "R32")
 					(unit 1)
 				)
@@
 		(in_pos_files yes)
 		(dnp no)
-		(property "Reference" "C36"
+		(property "Reference" "C42"
 			(at 96.012 133.858 0)
 			(show_name no)
@@
 			(project "FOC-driver"
 				(path "/1cfe65f9-f673-4819-b0fb-9ca652a1a340/f11b4b8c-1f7a-4164-8f83-b37924046d35"
-					(reference "C36")
+					(reference "C42")
 					(unit 1)
 				)
@@
 		(in_pos_files yes)
 		(dnp no)
-		(property "Reference" "D11"
+		(property "Reference" "D4"
 			(at 107.696 134.62 90)
 			(show_name no)
@@
 			(project "FOC-driver"
 				(path "/1cfe65f9-f673-4819-b0fb-9ca652a1a340/f11b4b8c-1f7a-4164-8f83-b37924046d35"
-					(reference "D11")
+					(reference "D4")
 					(unit 1)
 				)
@@
 		(in_pos_files yes)
 		(dnp no)
-		(property "Reference" "J19"
+		(property "Reference" "J5"
 			(at 99.06 57.15 0)
 			(show_name no)
@@
 			(project "FOC-driver"
 				(path "/1cfe65f9-f673-4819-b0fb-9ca652a1a340/f11b4b8c-1f7a-4164-8f83-b37924046d35"
-					(reference "J19")
+					(reference "J5")
 					(unit 1)
 				)
@@
 		(in_pos_files yes)
 		(dnp no)
-		(property "Reference" "C34"
+		(property "Reference" "C37"
 			(at 112.522 94.488 0)
 			(show_name no)
@@
 			(project "FOC-driver"
 				(path "/1cfe65f9-f673-4819-b0fb-9ca652a1a340/f11b4b8c-1f7a-4164-8f83-b37924046d35"
-					(reference "C34")
+					(reference "C37")
 					(unit 1)
 				)
@@
 		(in_pos_files yes)
 		(dnp no)
-		(property "Reference" "R31"
+		(property "Reference" "R33"
 			(at 158.75 95.504 90)
 			(show_name no)
@@
 			(project "FOC-driver"
 				(path "/1cfe65f9-f673-4819-b0fb-9ca652a1a340/f11b4b8c-1f7a-4164-8f83-b37924046d35"
-					(reference "R31")
+					(reference "R33")
 					(unit 1)
 				)
@@
 		(dnp yes)
 		(fields_autoplaced yes)
-		(property "Reference" "C40"
+		(property "Reference" "C46"
 			(at 116.84 54.9909 0)
 			(show_name no)
@@
 			(project "FOC-driver"
 				(path "/1cfe65f9-f673-4819-b0fb-9ca652a1a340/f11b4b8c-1f7a-4164-8f83-b37924046d35"
-					(reference "C40")
+					(reference "C46")
 					(unit 1)
 				)
@@
 		(in_pos_files yes)
 		(dnp no)
-		(property "Reference" "C35"
+		(property "Reference" "C41"
 			(at 57.912 135.128 0)
 			(show_name no)
@@
 			(project "FOC-driver"
 				(path "/1cfe65f9-f673-4819-b0fb-9ca652a1a340/f11b4b8c-1f7a-4164-8f83-b37924046d35"
-					(reference "C35")
+					(reference "C41")
 					(unit 1)
 				)
@@
 		(in_pos_files yes)
 		(dnp no)
-		(property "Reference" "L3"
+		(property "Reference" "L1"
 			(at 162.814 85.09 90)
 			(show_name no)
@@
 			(project "FOC-driver"
 				(path "/1cfe65f9-f673-4819-b0fb-9ca652a1a340/f11b4b8c-1f7a-4164-8f83-b37924046d35"
-					(reference "L3")
+					(reference "L1")
 					(unit 1)
 				)
@@
 		(in_pos_files yes)
 		(dnp no)
-		(property "Reference" "C29"
+		(property "Reference" "C38"
 			(at 125.222 94.488 0)
 			(show_name no)
@@
 			(project "FOC-driver"
 				(path "/1cfe65f9-f673-4819-b0fb-9ca652a1a340/f11b4b8c-1f7a-4164-8f83-b37924046d35"
-					(reference "C29")
+					(reference "C38")
 					(unit 1)
 				)
@@
 		(dnp no)
 		(fields_autoplaced yes)
-		(property "Reference" "U6"
+		(property "Reference" "U8"
 			(at 80.01 124.46 0)
 			(show_name no)
@@
 			(project "FOC-driver"
 				(path "/1cfe65f9-f673-4819-b0fb-9ca652a1a340/f11b4b8c-1f7a-4164-8f83-b37924046d35"
-					(reference "U6")
+					(reference "U8")
 					(unit 1)
 				)
@@
 		(in_pos_files yes)
 		(dnp no)
-		(property "Reference" "R39"
+		(property "Reference" "R35"
 			(at 100.33 127 90)
 			(show_name no)
@@
 			(project "FOC-driver"
 				(path "/1cfe65f9-f673-4819-b0fb-9ca652a1a340/f11b4b8c-1f7a-4164-8f83-b37924046d35"
-					(reference "R39")
+					(reference "R35")
 					(unit 1)
 				)
@@
 		(in_pos_files yes)
 		(dnp no)
-		(property "Reference" "R36"
+		(property "Reference" "R34"
 			(at 68.58 137.922 90)
 			(show_name no)
@@
 			(project "FOC-driver"
 				(path "/1cfe65f9-f673-4819-b0fb-9ca652a1a340/f11b4b8c-1f7a-4164-8f83-b37924046d35"
-					(reference "R36")
+					(reference "R34")
 					(unit 1)
 				)
@@
 		(in_pos_files yes)
 		(dnp no)
-		(property "Reference" "R33"
+		(property "Reference" "R30"
 			(at 68.072 89.154 0)
 			(show_name no)
@@
 			(project "FOC-driver"
 				(path "/1cfe65f9-f673-4819-b0fb-9ca652a1a340/f11b4b8c-1f7a-4164-8f83-b37924046d35"
-					(reference "R33")
-					(unit 1)
-				)
+					(reference "R30")
+					(unit 1)
+				)

Commit message: commit
Parts:
- added R41: 10k, Resistor_SMD:R_0402_1005Metric, symbol Device:R_Small
- J5: footprint addons:2p WireSolder 1.5mmID_2.5mmOD -> addons:2p WireSolder 1.3mmID_2mmOD
Connections:
- net GND: now also U7.2 (GND); no longer U7.1 (GND)
- net at C39.1, L1.1: now also U7.6 (SW); no longer U7.2 (SW)
- net at C39.2: now also U7.1 (CB); no longer U7.6 (CB)
- net at C37.1, C38.1, FB2.2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: now also R41.2; no longer U7.3 (VIN)
- net at R32.1, R33.1: now also U7.3 (FB); no longer U7.4 (FB)
- new net: R41.1, U7.4 (EN)
Other:
- moved on the sheet: C39, C40, L1, R32, R33, U7
