File: Kicad/untitled.kicad_sch (KiCad schematic)
At the start: 25 parts, among them J18 Thermistor, U4 STM32G473RCTx, U5 AS5047P, Y1 24MHz

Commit message: hw(stm32): changed MCU to STM32G431CBTx since opamps unused.
Parts:
- removed C4: 100n, Capacitor_SMD:C_0402_1005Metric, symbol Device:C_Small
- removed U4: STM32G473RCTx, Package_QFP:LQFP-64_10x10mm_P0.5mm, symbol MCU_ST_STM32G4:STM32G473RCTx
- added U11: STM32G431C8Tx, Package_QFP:LQFP-48_7x7mm_P0.5mm, symbol MCU_ST_STM32G4:STM32G431C8Tx
Connections:
- net +3.3V: now also U11.1 (VBAT), U11.24 (VDD), U11.36 (VDD), U11.48 (VDD)
- net +3.3VA: now also U11.20 (VREF+), U11.21 (VDDA)
- net ENC_CS: now also U11.43 (PB6)
- net FDCAN1_Rx: now also U11.45 (PB8)
- net FDCAN1_Tx: now also U11.46 (PB9)
- net GND: now also U11.19 (VSSA), U11.23 (VSS), U11.35 (VSS), U11.47 (VSS)
- net HIN_A: now also U11.30 (PA8)
- net HIN_B: now also U11.31 (PA9)
- net HIN_C: now also U11.32 (PA10)
- net I2C1_SCL: now also U11.39 (PA15)
- net I2C1_SDA: now also U11.44 (PB7)
- net ISENSE_A: now also U11.8 (PA0)
- net ISENSE_B: now also U11.9 (PA1)
- net ISENSE_C: now also U11.14 (PA6)
- net MOTOR_TEMP: now also U11.26 (PB12)
- net NLIN_A: now also U11.2 (PC13)
- net NLIN_B: now also U11.16 (PB0)
- net NLIN_C: now also U11.17 (PB1)
- net NRST: now also U11.7 (PG10)
- net SPI1_CLK: now also U11.13 (PA5)
- net SPI1_MISO: now also U11.41 (PB4)
- net SPI1_MOSI: now also U11.42 (PB5)
- net SWCLK: now also U11.38 (PA14)
- net SWDIO: now also U11.37 (PA13)
- net USB_D+: now also U11.34 (PA12)
- net USB_D-: now also U11.33 (PA11)
- net VSENSE_A: now also U11.10 (PA2)
- net VSENSE_B: now also U11.11 (PA3)
- net VSENSE_C: now also U11.28 (PB14)
- net VSENSE_SUP: now also U11.15 (PA7)
- net nFAULT: now also U11.27 (PB13)
- net nSLEEP: now also U11.25 (PB11)
- net at R38.2: now also U11.22 (PB10)
- net at C10.1, Y1.1: now also U11.5 (PF0)
- net at C11.1, Y1.3: now also U11.6 (PF1)
- no-connect marks 25 -> 12
Other:
- moved on the sheet: C5, C6, C7, C8, D10, FB1, R38

Commit message: hw(pcb-sch): rename component ref & pcb manufacturing capability
Parts:
- renumbered C5 to C1, C27 to C10, C10 to C11, C11 to C12, C44 to C13, C17 to C14, C3 to C2, C2 to C3, C1 to C4, C15 to C5, C8 to C7, C7 to C8, C26 to C9, D10 to D1, J18 to J1, R37 to R1, R38 to R2, R40 to R3, R41 to R4
Changed lines of the file:
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@@
 		(in_pos_files yes)
 		(dnp no)
-		(property "Reference" "J18"
+		(property "Reference" "J1"
 			(at 204.47 63.5 0)
 			(show_name no)
@@
 			(project "FOC-driver"
 				(path "/1cfe65f9-f673-4819-b0fb-9ca652a1a340/0fd646cd-1189-4702-9277-d0a075d515a1"
-					(reference "J18")
+					(reference "J1")
 					(unit 1)
 				)
@@
 		(dnp no)
 		(fields_autoplaced yes)
-		(property "Reference" "C5"
+		(property "Reference" "C1"
 			(at 57.15 49.5362 0)
 			(show_name no)
@@
 			(project "FOC-driver"
 				(path "/1cfe65f9-f673-4819-b0fb-9ca652a1a340/0fd646cd-1189-4702-9277-d0a075d515a1"
-					(reference "C5")
+					(reference "C1")
 					(unit 1)
 				)
@@
 		(in_pos_files yes)
 		(dnp no)
-		(property "Reference" "R38"
+		(property "Reference" "R2"
 			(at 67.056 123.698 90)
 			(show_name no)
@@
 			(project "FOC-driver"
 				(path "/1cfe65f9-f673-4819-b0fb-9ca652a1a340/0fd646cd-1189-4702-9277-d0a075d515a1"
-					(reference "R38")
+					(reference "R2")
 					(unit 1)
 				)
@@
 		(in_pos_files yes)
 		(dnp no)
-		(property "Reference" "R41"
+		(property "Reference" "R4"
 			(at 219.964 55.118 90)
 			(show_name no)
@@
 			(project "FOC-driver"
 				(path "/1cfe65f9-f673-4819-b0fb-9ca652a1a340/0fd646cd-1189-4702-9277-d0a075d515a1"
-					(reference "R41")
+					(reference "R4")
 					(unit 1)
 				)
@@
 		(in_pos_files yes)
 		(dnp no)
-		(property "Reference" "C10"
+		(property "Reference" "C11"
 			(at 40.894 96.52 0)
 			(show_name no)
@@
 			(project "FOC-driver"
 				(path "/1cfe65f9-f673-4819-b0fb-9ca652a1a340/0fd646cd-1189-4702-9277-d0a075d515a1"
-					(reference "C10")
+					(reference "C11")
 					(unit 1)
 				)
@@
 		(dnp no)
 		(fields_autoplaced yes)
-		(property "Reference" "C15"
+		(property "Reference" "C5"
 			(at 93.98 49.5362 0)
 			(show_name no)
@@
 			(project "FOC-driver"
 				(path "/1cfe65f9-f673-4819-b0fb-9ca652a1a340/0fd646cd-1189-4702-9277-d0a075d515a1"
-					(reference "C15")
+					(reference "C5")
 					(unit 1)
 				)
@@
 		(dnp no)
 		(fields_autoplaced yes)
-		(property "Reference" "C11"
+		(property "Reference" "C12"
 			(at 64.77 96.5262 0)
 			(show_name no)
@@
 			(project "FOC-driver"
 				(path "/1cfe65f9-f673-4819-b0fb-9ca652a1a340/0fd646cd-1189-4702-9277-d0a075d515a1"
-					(reference "C11")
+					(reference "C12")
 					(unit 1)
 				)
@@
 		(dnp no)
 		(fields_autoplaced yes)
-		(property "Reference" "C26"
+		(property "Reference" "C9"
 			(at 77.4763 59.69 90)
 			(show_name no)
@@
 			(project "FOC-driver"
 				(path "/1cfe65f9-f673-4819-b0fb-9ca652a1a340/0fd646cd-1189-4702-9277-d0a075d515a1"
-					(reference "C26")
+					(reference "C9")
 					(unit 1)
 				)
@@
 		(in_pos_files yes)
 		(dnp no)
-		(property "Reference" "R37"
+		(property "Reference" "R1"
 			(at 66.802 66.294 0)
 			(show_name no)
@@
 			(project "FOC-driver"
 				(path "/1cfe65f9-f673-4819-b0fb-9ca652a1a340/0fd646cd-1189-4702-9277-d0a075d515a1"
-					(reference "R37")
+					(reference "R1")
 					(unit 1)
 				)
@@
 		(dnp no)
 		(fields_autoplaced yes)
-		(property "Reference" "C2"
+		(property "Reference" "C3"
 			(at 76.2 49.5362 0)
 			(show_name no)
@@
 			(project "FOC-driver"
 				(path "/1cfe65f9-f673-4819-b0fb-9ca652a1a340/0fd646cd-1189-4702-9277-d0a075d515a1"
-					(reference "C2")
+					(reference "C3")
 					(unit 1)
 				)
@@
 		(dnp no)
 		(fields_autoplaced yes)
-		(property "Reference" "C1"
+		(property "Reference" "C4"
 			(at 85.09 49.5362 0)
 			(show_name no)
@@
 			(project "FOC-driver"
 				(path "/1cfe65f9-f673-4819-b0fb-9ca652a1a340/0fd646cd-1189-4702-9277-d0a075d515a1"
-					(reference "C1")
+					(reference "C4")
 					(unit 1)
 				)
@@
 		(in_pos_files yes)
 		(dnp no)
-		(property "Reference" "R40"
+		(property "Reference" "R3"
 			(at 197.104 55.118 90)
 			(show_name no)
@@
 			(project "FOC-driver"
 				(path "/1cfe65f9-f673-4819-b0fb-9ca652a1a340/0fd646cd-1189-4702-9277-d0a075d515a1"
-					(reference "R40")
+					(reference "R3")
 					(unit 1)
 				)
@@
 		(dnp no)
 		(fields_autoplaced yes)
-		(property "Reference" "C8"
+		(property "Reference" "C7"
 			(at 129.54 49.5362 0)
 			(show_name no)
@@
 			(project "FOC-driver"
 				(path "/1cfe65f9-f673-4819-b0fb-9ca652a1a340/0fd646cd-1189-4702-9277-d0a075d515a1"
-					(reference "C8")
+					(reference "C7")
 					(unit 1)
 				)
@@
 		(dnp no)
 		(fields_autoplaced yes)
-		(property "Reference" "C7"
+		(property "Reference" "C8"
 			(at 143.51 49.5362 0)
 			(show_name no)
@@
 			(project "FOC-driver"
 				(path "/1cfe65f9-f673-4819-b0fb-9ca652a1a340/0fd646cd-1189-4702-9277-d0a075d515a1"
-					(reference "C7")
+					(reference "C8")
 					(unit 1)
 				)
@@
 		(dnp no)
 		(fields_autoplaced yes)
-		(property "Reference" "C3"
+		(property "Reference" "C2"
 			(at 67.31 49.5362 0)
 			(show_name no)
@@
 			(project "FOC-driver"
 				(path "/1cfe65f9-f673-4819-b0fb-9ca652a1a340/0fd646cd-1189-4702-9277-d0a075d515a1"
-					(reference "C3")
+					(reference "C2")
 					(unit 1)
 				)
@@
 		(in_pos_files yes)
 		(dnp no)
-		(property "Reference" "D10"
+		(property "Reference" "D1"
 			(at 59.944 123.19 90)
 			(show_name no)
@@
 			(project "FOC-driver"
 				(path "/1cfe65f9-f673-4819-b0fb-9ca652a1a340/0fd646cd-1189-4702-9277-d0a075d515a1"
-					(reference "D10")
+					(reference "D1")
 					(unit 1)
 				)
@@
 		(dnp no)
 		(fields_autoplaced yes)
-		(property "Reference" "C44"
+		(property "Reference" "C13"
 			(at 214.63 62.2235 0)
 			(show_name no)
@@
 			(project "FOC-driver"
 				(path "/1cfe65f9-f673-4819-b0fb-9ca652a1a340/0fd646cd-1189-4702-9277-d0a075d515a1"
-					(reference "C44")
+					(reference "C13")
 					(unit 1)
 				)
@@
 		(dnp no)
 		(fields_autoplaced yes)
-		(property "Reference" "C17"
+		(property "Reference" "C14"
 			(at 196.85 125.7362 0)
 			(show_name no)
@@
 			(project "FOC-driver"
 				(path "/1cfe65f9-f673-4819-b0fb-9ca652a1a340/0fd646cd-1189-4702-9277-d0a075d515a1"
-					(reference "C17")
+					(reference "C14")
 					(unit 1)
 				)
@@
 		(dnp no)
 		(fields_autoplaced yes)
-		(property "Reference" "C27"
+		(property "Reference" "C10"
 			(at 64.77 73.6535 0)
 			(show_name no)
@@
 			(project "FOC-driver"
 				(path "/1cfe65f9-f673-4819-b0fb-9ca652a1a340/0fd646cd-1189-4702-9277-d0a075d515a1"
-					(reference "C27")
+					(reference "C10")
 					(unit 1)
 				)

Commit message: hw(pcb): initial grouping + layout guidlines
Parts:
- C9: footprint Capacitor_SMD:C_01005_0402Metric -> Capacitor_SMD:C_0402_1005Metric
- renumbered U11 to U1, U5 to U2
Connections:
- net HSE_IN: now reaches C11.1, U1.5 (PF0), Y1.1
- net HSE_OUT: now reaches C12.1, U1.6 (PF1), Y1.3
Other:
- moved on the sheet: D1, R2

Commit message: commit
Parts:
- added R40: 10k, Resistor_SMD:R_0402_1005Metric, symbol Device:R_Small
- R3, R4: footprint Resistor_SMD:R_01005_0402Metric -> Resistor_SMD:R_0402_1005Metric
Connections:
- net +3.3V: now also R40.1
- net ENC_CS: now also R40.2
- net +5V: no longer names the net of U2.11 (VDD)
- no-connect marks 12 -> 13
Other:
- moved on the sheet: C14, U2
